File: Universal_Modern_PSU_12V_Input/Universal_Modern_PSU_12V_Input.kicad_sch (KiCad schematic)
At the start: 27 parts, among them J1 +12VDC Input, J2 Power Output, Q1 SUP53P06-20-E3, Q2 SUP53P06-20-E3, U1 DFR0831, U2 NKE1212SC, U3 R-78CK5.0-0.5

Commit message: Fix pin order of output header
Parts:
- J2: footprint Clueless_Engineer:640445-5 -> Clueless_Engineer:640445-6
Connections:
- net +12V_{IN}: now also J2.2 (Pin_2); no longer J2.4 (Pin_4)
- net -5V_{OUT}: now also J2.3 (Pin_3); no longer J2.2 (Pin_2)
- net GND: now also J2.4 (Pin_4); no longer J2.3 (Pin_3)
Changed lines of the file:
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@@
 			)
 		)
-		(property "Footprint" "Clueless_Engineer:640445-5"
+		(property "Footprint" "Clueless_Engineer:640445-6"
 			(at 257.81 93.98 0)
 			(hide yes)
